Commit message: Config turtlebot3 to use node

File: urdf/gazebo_specific.urdf.xacro (robot description, xacro)
@@ -1,4 +1,4 @@
 <?xml version="1.0"?>
-<robot xmlns:xacro="http://ros.org/wiki/xacro" name="noah_wheel">
+<robot xmlns:xacro="http://ros.org/wiki/xacro" name="turtlebot3">
 	<xacro:macro name="gazebo_specific" params="frame_prefix topic_prefix">
     <gazebo>

File: urdf/turtlebot3_waffle.urdf.xacro (robot description, xacro)
@@ -71,4 +71,7 @@
     </inertial>
   </link>
+  <gazebo reference="base_link">
+    <material>Gazebo/Gray</material>
+  </gazebo>
   <joint name="wheel_left_joint" type="continuous">
     <parent link="base_link"/>
